File: Solder practice heart.kicad_pcb (KiCad board)
At the start: 2 copper layers, 101.6 x 101.6 mm, 26 parts

Commit message: Redone PCB, added Gerbers
Parts:
- moved BAT2 16.4 mm to (176.5, 138.4)
- moved BAT1 16.0 mm to (127.0, 138.4)
- moved LED15 2.39 mm to (132.6, 116.8), turned to 0 degrees
- moved LED6 1.81 mm to (180.8, 81.0), turned to 0 degrees
- moved LED9 1.53 mm to (151.8, 87.9), turned to 0 degrees
- moved LED1 1.34 mm to (153.1, 133.2), turned to 90 degrees
Routing:
- net Net-(LED1-K): track 0.00 -> 15.5 mm
- net Net-(LED7-K): track 0.00 -> 15.4 mm
- net Net-(LED13-K): track 0.00 -> 14.4 mm
- net Net-(LED15-K): track 0.00 -> 14.3 mm
- net Net-(LED5-K): track 0.00 -> 13.8 mm
- net Net-(LED3-K): track 0.00 -> 13.8 mm
- net Net-(LED11-K): track 0.00 -> 13.2 mm
- net Net-(LED10-A): track 0.00 -> 12.2 mm
- net Net-(LED6-K): track 0.00 -> 6.75 mm
- net Net-(LED4-K): track 0.00 -> 6.20 mm
- net Net-(LED10-K): track 0.00 -> 6.00 mm
- net Net-(LED12-K): track 0.00 -> 5.58 mm
- net Net-(LED16-K): track 0.00 -> 5.29 mm
- net Net-(LED2-K): track 0.00 -> 4.17 mm
- net Net-(LED14-K): track 0.00 -> 4.13 mm
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Other:
- board size 101.6 x 101.6 mm -> 83.8 x 101.6 mm
- board text removed: "Solder practice heart (C) 2025 Stefan Gofferje CC-BY-SA 4.0"

Commit message: Forgot one track...
Routing:
- net Net-(BAT1-Pad2): track 0.00 -> 28.7 mm
Changed lines of the file:
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@@
 		(tags "LED diameter 5.0mm 2 pins")
 		(property "Reference" "LED15"
-			(at 1.27 -3.96 360)
+			(at 1.27 -3.96 0)
 			(layer "F.SilkS")
 			(effects
@@
 		)
 		(property "Value" "LED_5mm_Red"
-			(at 1.27 3.96 360)
+			(at 1.27 3.96 0)
 			(layer "F.Fab")
 			(hide yes)
@@
 		)
 		(property "Footprint" "PCM_LED_THT_AKL:LED_D5.0mm"
-			(at 0 0 360)
+			(at 0 0 0)
 			(layer "F.Fab")
 			(hide yes)
@@
 		)
 		(property "Datasheet" ""
-			(at 0 0 360)
+			(at 0 0 0)
 			(layer "F.Fab")
 			(hide yes)
@@
 		)
 		(property "Description" "Red LED, 5mm THT, Alternate KiCad Library"
-			(at 0 0 360)
+			(at 0 0 0)
 			(layer "F.Fab")
 			(hide yes)
@@
 		)
 		(fp_text user "${REFERENCE}"
-			(at 1.25 0 360)
+			(at 1.25 0 0)
 			(layer "F.Fab")
 			(effects
@@
 		(tags "LED diameter 5.0mm 2 pins")
 		(property "Reference" "LED9"
-			(at 1.27 -3.96 360)
+			(at 1.27 -3.96 0)
 			(layer "F.SilkS")
 			(effects
@@
 		)
 		(property "Value" "LED_5mm_Red"
-			(at 1.27 3.96 360)
+			(at 1.27 3.96 0)
 			(layer "F.Fab")
 			(hide yes)
@@
 		)
 		(property "Footprint" "PCM_LED_THT_AKL:LED_D5.0mm"
-			(at 0 0 360)
+			(at 0 0 0)
 			(layer "F.Fab")
 			(hide yes)
@@
 		)
 		(property "Datasheet" ""
-			(at 0 0 360)
+			(at 0 0 0)
 			(layer "F.Fab")
 			(hide yes)
@@
 		)
 		(property "Description" "Red LED, 5mm THT, Alternate KiCad Library"
-			(at 0 0 360)
+			(at 0 0 0)
 			(layer "F.Fab")
 			(hide yes)
@@
 		)
 		(fp_text user "${REFERENCE}"
-			(at 1.25 0 360)
+			(at 1.25 0 0)
 			(layer "F.Fab")
 			(effects
@@
 		(tags "LED diameter 5.0mm 2 pins")
 		(property "Reference" "LED6"
-			(at 1.27 -3.96 360)
+			(at 1.27 -3.96 0)
 			(layer "F.SilkS")
 			(effects
@@
 		)
 		(property "Value" "LED_5mm_Red"
-			(at 1.27 3.96 360)
+			(at 1.27 3.96 0)
 			(layer "F.Fab")
 			(hide yes)
@@
 		)
 		(property "Footprint" "PCM_LED_THT_AKL:LED_D5.0mm"
-			(at 0 0 360)
+			(at 0 0 0)
 			(layer "F.Fab")
 			(hide yes)
@@
 		)
 		(property "Datasheet" ""
-			(at 0 0 360)
+			(at 0 0 0)
 			(layer "F.Fab")
 			(hide yes)
@@
 		)
 		(property "Description" "Red LED, 5mm THT, Alternate KiCad Library"
-			(at 0 0 360)
+			(at 0 0 0)
 			(layer "F.Fab")
 			(hide yes)
@@
 		)
 		(fp_text user "${REFERENCE}"
-			(at 1.25 0 360)
+			(at 1.25 0 0)
 			(layer "F.Fab")
 			(effects
@@
 	)
 	(segment
+		(start 137.4 138.43)
+		(end 166.13 138.43)
+		(width 0.8)
+		(layer "B.Cu")
+		(net 2)
+	)
+	(segment

Commit message: Add license text to PCB silkscreen Update Readme
Other:
- board text added: "Heart shaped solder practice PCB for kids (C) 2025 Stefan Gofferje License: CC-BY-SA 4.0"
- board text added: "This PCB was built by: On:"
Changed lines of the file:
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@@
 		(layer "Edge.Cuts")
+	)
+	(gr_text "This PCB was built by:\n\n\n\n\n\nOn:"
+		(at 165.664287 107.95 0)
+		(layer "B.SilkS")
+		(effects
+			(font
+				(size 1.5 1.5)
+				(thickness 0.3)
+				(bold yes)
+			)
+			(justify left bottom mirror)
+		)
+	)
+	(gr_text "Heart shaped solder practice PCB for kids\n(C) 2025 Stefan Gofferje\nLicense: CC-BY-SA 4.0"
+		(at 152.4 66.860749 0)
+		(layer "B.SilkS")
+		(effects
+			(font
+				(size 1.5 1.5)
+				(thickness 0.3)
+				(bold yes)
+			)
+			(justify bottom mirror)
+		)
 	)
 	(segment
